Commit message: Change my bot to use vacuum cleaner model

File: urdf/my_bot.xacro (robot description, xacro)
@@ -9,66 +9,72 @@
   </joint>
   <link name='chassis'>
-    <pose>0 0 0.1 0 0 0</pose>
+    <pose>0 0 0.071 0 0 0</pose>
     <inertial>
-      <mass value="15.0"/>
-      <origin xyz="0.0 0 0" rpy=" 0 0 0"/>
+      <mass value="5.0"/>
+      <origin xyz="0 0 0" rpy="0 0 0"/>
       <inertia
-          ixx="0.1" ixy="0" ixz="0"
-          iyy="0.1" iyz="0"
-          izz="0.1"
+          ixx="0.08229" ixy="0" ixz="0"
+          iyy="0.08229" iyz="0"
+          izz="0.15625"
       />
     </inertial>
     <collision name='collision'>
-      <origin xyz="0 0 0" rpy=" 0 0 0"/>
+      <origin xyz="0 0 0" rpy="0 0 0"/>
       <geometry>
-        <box size=".4 .2 .1"/>
+        <cylinder radius="0.25" length="0.1"/>
       </geometry>
     </collision>
     <visual name='chassis_visual'>
-      <origin xyz="0 0 0" rpy=" 0 0 0"/>
+      <origin xyz="0 0 0" rpy="0 0 0"/>
       <geometry>
-        <box size=".4 .2 .1"/>
-      </geometry>
-    </visual>
-    <collision name='back_caster_collision'>
-      <origin xyz="-0.15 0 -0.05" rpy=" 0 0 0"/>
-      <geometry>
-        <sphere radius="0.0499"/>
-      </geometry>
-    </collision>
-    <visual name='back_caster_visual'>
-      <origin xyz="-0.15 0 -0.05" rpy=" 0 0 0"/>
-      <geometry>
-        <sphere radius="0.05"/>
-      </geometry>
-    </visual>
-    <collision name='front_caster_collision'>
-      <origin xyz="0.15 0 -0.05" rpy=" 0 0 0"/>
-      <geometry>
-        <sphere radius="0.0499"/>
-      </geometry>
-    </collision>
-    <visual name='front_caster_visual'>
-      <origin xyz="0.15 0 -0.05" rpy=" 0 0 0"/>
-      <geometry>
-        <sphere radius="0.05"/>
+        <cylinder radius="0.25" length="0.1"/>
       </geometry>
     </visual>
   </link>
+  <link name='caster'>
+    <pose>0 0 0 0 0 0</pose>
+    <inertial>
+      <mass value="1.0"/>
+      <origin xyz="0 0 0" rpy="0 0 0"/>
+      <inertia
+          ixx="0.0267" ixy="0" ixz="0"
+          iyy="0.0267" iyz="0"
+          izz="0.0267"
+      />
+    </inertial>
+    <collision name='caster_collision'>
+      <origin xyz="0 0 0" rpy="0 0 0"/>
+      <geometry>
+        <sphere radius="0.02"/>
+      </geometry>
+    </collision>
+    <visual name='caster_visual'>
+      <origin xyz="0 0 0" rpy="0 0 0"/>
+      <geometry>
+        <sphere radius="0.02"/>
+      </geometry>
+    </visual>
+  </link>
+  <joint type="fixed" name="caster_joint">
+    <origin xyz="0.21 0 -0.05" rpy="0 0 0"/>
+    <child link="caster"/>
+    <parent link="chassis"/>
+    <dynamics damping="0.0" friction="0.0"/>
+  </joint>
   <link name='left_wheel'>
     <pose>0 0 0 0 0 0</pose>
     <inertial>
-      <mass value="5.0"/>
+      <mass value="1.0"/>
       <origin xyz="0 0 0" rpy="0 1.5707 1.5707"/>
       <inertia
-          ixx="0.1" ixy="0" ixz="0"
-          iyy="0.1" iyz="0"
-          izz="0.1"
+          ixx="0.0133" ixy="0" ixz="0"
+          iyy="0.0133" iyz="0"
+          izz="0.02"
       />
     </inertial>
-    <collision name='collision'>
+    <collision name='left_collision'>
       <origin xyz="0 0 0" rpy="0 1.5707 1.5707"/>
       <geometry>
-        <cylinder radius="0.1" length="0.05"/>
+        <cylinder radius="0.02" length="0.02"/>
       </geometry>
     </collision>
@@ -76,10 +82,10 @@
       <origin xyz="0 0 0" rpy="0 1.5707 1.5707"/>
       <geometry>
-        <cylinder radius="0.1" length="0.05"/>
+        <cylinder radius="0.02" length="0.02"/>
       </geometry>
     </visual>
   </link>
   <joint type="continuous" name="left_wheel_hinge">
-    <origin xyz="0 0.15 0" rpy="0 0 0"/>
+    <origin xyz="-0.15 0.15 -0.05" rpy="0 0 0"/>
     <child link="left_wheel"/>
     <parent link="chassis"/>
@@ -91,16 +97,16 @@
     <pose>0 0 0 0 0 0</pose>
     <inertial>
-      <mass value="5.0"/>
+      <mass value="1.0"/>
       <origin xyz="0 0 0" rpy="0 1.5707 1.5707"/>
       <inertia
-          ixx="0.1" ixy="0" ixz="0"
-          iyy="0.1" iyz="0"
-          izz="0.1"
-      />
+          ixx="0.0133" ixy="0" ixz="0"
+          iyy="0.0133" iyz="0"
+          izz="0.02"
+     />
     </inertial>
-    <collision name='collision'>
+    <collision name='right_collision'>
       <origin xyz="0 0 0" rpy="0 1.5707 1.5707"/>
       <geometry>
-        <cylinder radius="0.1" length="0.05"/>
+        <cylinder radius="0.02" length="0.02"/>
       </geometry>
     </collision>
@@ -108,25 +114,25 @@
       <origin xyz="0 0 0" rpy="0 1.5707 1.5707"/>
       <geometry>
-        <cylinder radius="0.1" length="0.05"/>
+        <cylinder radius="0.02" length="0.02"/>
       </geometry>
     </visual>
   </link>
   <joint type="continuous" name="right_wheel_hinge">
-    <origin xyz="0 -0.15 0" rpy="0 0 0"/>
+    <origin xyz="-0.15 -0.15 -0.05" rpy="0 0 0"/>
     <child link="right_wheel"/>
     <parent link="chassis"/>
     <axis xyz="0 1 0" rpy="0 0 0"/>
     <limit effort="10000" velocity="1000"/>
-    <dynamics damping="1.0" friction="1.0"/>
+    <dynamics damping="10.0" friction="10.0"/>
   </joint>
   <link name='camera'>
     <pose>0 0 0 0 0 0</pose>
     <inertial>
-      <mass value="0.1"/>
+      <mass value="0.5"/>
       <origin xyz="0 0 0" rpy="0 0 0"/>
       <inertia
-          ixx="1e-6" ixy="0" ixz="0"
-          iyy="1e-6" iyz="0"
-          izz="1e-6"
+          ixx="0.000208" ixy="0" ixz="0"
+          iyy="0.000208" iyz="0"
+          izz="0.000208"
       />
     </inertial>
@@ -145,5 +151,5 @@
   </link>
   <joint type="fixed" name="camera_joint">
-    <origin xyz="0.2 0 0" rpy="0 0 0"/>
+    <origin xyz="0.24 0 0" rpy="0 0 0"/>
     <child link="camera"/>
     <parent link="chassis"/>
@@ -152,10 +158,10 @@
     <pose>0 0 0 0 0 0</pose>
     <inertial>
-      <mass value="0.1"/>
+      <mass value="1.0"/>
       <origin xyz="0 0 0" rpy="0 0 0"/>
       <inertia
-          ixx="1e-6" ixy="0" ixz="0"
-          iyy="1e-6" iyz="0"
-          izz="1e-6"
+          ixx="0.001667" ixy="0" ixz="0"
+          iyy="0.001667" iyz="0"
+          izz="0.001667"
       />
     </inertial>
@@ -174,5 +180,5 @@
   </link>
   <joint type="fixed" name="hokuyo_joint">
-    <origin xyz=".15 0 .1" rpy="0 0 0"/>
+    <origin xyz="0 0 0.1" rpy="0 0 0"/>
     <child link="hokuyo"/>
     <parent link="chassis"/>

Commit message: Fix very slow motion

File: urdf/my_bot.xacro (robot description, xacro)
@@ -11,5 +11,5 @@
     <pose>0 0 0.071 0 0 0</pose>
     <inertial>
-      <mass value="5.0"/>
+      <mass value="10.0"/>
       <origin xyz="0 0 0" rpy="0 0 0"/>
       <inertia
@@ -151,5 +151,5 @@
   </link>
   <joint type="fixed" name="camera_joint">
-    <origin xyz="0.24 0 0" rpy="0 0 0"/>
+    <origin xyz="0.25 0 0" rpy="0 0 0"/>
     <child link="camera"/>
     <parent link="chassis"/>

Commit message: Make my_bot achieve the goal

File: urdf/my_bot.xacro (robot description, xacro)
@@ -22,5 +22,5 @@
       <origin xyz="0 0 0" rpy="0 0 0"/>
       <geometry>
-        <cylinder radius="0.25" length="0.1"/>
+        <cylinder radius="0.2" length="0.1"/>
       </geometry>
     </collision>
@@ -28,5 +28,5 @@
       <origin xyz="0 0 0" rpy="0 0 0"/>
       <geometry>
-        <cylinder radius="0.25" length="0.1"/>
+        <cylinder radius="0.2" length="0.1"/>
       </geometry>
     </visual>
@@ -57,5 +57,5 @@
   </link>
   <joint type="fixed" name="caster_joint">
-    <origin xyz="0.21 0 -0.05" rpy="0 0 0"/>
+    <origin xyz="0.16 0 -0.05" rpy="0 0 0"/>
     <child link="caster"/>
     <parent link="chassis"/>
@@ -87,10 +87,10 @@
   </link>
   <joint type="continuous" name="left_wheel_hinge">
-    <origin xyz="-0.15 0.15 -0.05" rpy="0 0 0"/>
+    <origin xyz="0.0 0.15 -0.05" rpy="0 0 0"/>
     <child link="left_wheel"/>
     <parent link="chassis"/>
     <axis xyz="0 1 0" rpy="0 0 0"/>
     <limit effort="10000" velocity="1000"/>
-    <dynamics damping="1.0" friction="1.0"/>
+    <dynamics damping="0.1" friction="0.1"/>
   </joint>
   <link name='right_wheel'>
@@ -119,20 +119,20 @@
   </link>
   <joint type="continuous" name="right_wheel_hinge">
-    <origin xyz="-0.15 -0.15 -0.05" rpy="0 0 0"/>
+    <origin xyz="0.0 -0.15 -0.05" rpy="0 0 0"/>
     <child link="right_wheel"/>
     <parent link="chassis"/>
     <axis xyz="0 1 0" rpy="0 0 0"/>
     <limit effort="10000" velocity="1000"/>
-    <dynamics damping="10.0" friction="10.0"/>
+    <dynamics damping="0.1" friction="0.1"/>
   </joint>
   <link name='camera'>
     <pose>0 0 0 0 0 0</pose>
     <inertial>
-      <mass value="0.5"/>
+      <mass value="5.0"/>
       <origin xyz="0 0 0" rpy="0 0 0"/>
       <inertia
-          ixx="0.000208" ixy="0" ixz="0"
-          iyy="0.000208" iyz="0"
-          izz="0.000208"
+          ixx="0.00208" ixy="0" ixz="0"
+          iyy="0.00208" iyz="0"
+          izz="0.00208"
       />
     </inertial>
@@ -151,5 +151,5 @@
   </link>
   <joint type="fixed" name="camera_joint">
-    <origin xyz="0.25 0 0" rpy="0 0 0"/>
+    <origin xyz="0.20 0 0" rpy="0 0 0"/>
     <child link="camera"/>
     <parent link="chassis"/>
@@ -180,5 +180,5 @@
   </link>
   <joint type="fixed" name="hokuyo_joint">
-    <origin xyz="0 0 0.1" rpy="0 0 0"/>
+    <origin xyz="0 0 0.08" rpy="0 0 0"/>
     <child link="hokuyo"/>
     <parent link="chassis"/>
